Commit message: fixed bugs created generator version with and without prefixes (arg prefix cannot be empty)

File: sr_moveit_hand_config/config/shadowhand.srdf.xacro (robot description, xacro)
@@ -41,5 +41,4 @@
        <joint name="${prefix}${joint_prefix}J5" value="0" />
       </xacro:if>
-  </xacro:macro>
   </xacro:macro>
   <xacro:macro name="thumb_state_open" params="prefix is_lite">
