Commit message: Reverted xacro calls to indigo API Removed properties from inside macros Fixed tip_name when prefix

File: sr_moveit_hand_config/config/shadowhand.srdf.xacro (robot description, xacro)
@@ -23,14 +23,7 @@
     <joint name="${prefix}${joint_prefix}J2" />
     <joint name="${prefix}${joint_prefix}J1" />
-  </xacro:macro>
-  <xacro:macro name="fingerlinks" params="prefix link_prefix lf bio">
-    <xacro:if value="${bio}">
-      <xacro:property name="distal" value="biotac"/>
-      <xacro:property name="middle" value="adapter"/>
-    </xacro:if>
-    <xacro:unless value="${bio}">
-      <xacro:property name="distal" value="distal"/>
-      <xacro:property name="middle" value="middle"/>
-    </xacro:unless>
+    <joint name="${prefix}${joint_prefix}tip" />
+  </xacro:macro>
+  <xacro:macro name="fingerlinks" params="prefix link_prefix lf">
     <xacro:if value="${lf}">
       <!-- Little finger special case -->
@@ -49,11 +42,5 @@
     <joint name="${prefix}THJ1" />
   </xacro:macro>
-  <xacro:macro name="thumblinks" params="prefix bio" >
-    <xacro:if value="${bio}">
-      <xacro:property name="distal" value="biotac"/>
-    </xacro:if>
-    <xacro:unless value="${bio}">
-      <xacro:property name="distal" value="distal"/>
-    </xacro:unless>
+  <xacro:macro name="thumblinks" params="prefix" >
     <link name="${prefix}thbase" />
     <link name="${prefix}thproximal" />
@@ -109,13 +96,5 @@
     <passive_joint name="${prefix}virtual_joint" />
   </xacro:macro>
-  <xacro:macro name="finger_collisions" params="prefix link_prefix lf bio" >
-    <xacro:if value="${bio}">
-      <xacro:property name="distal" value="biotac"/>
-      <xacro:property name="middle" value="adapter"/>
-    </xacro:if>
-    <xacro:unless value="${bio}">
-      <xacro:property name="distal" value="distal"/>
-      <xacro:property name="middle" value="middle"/>
-    </xacro:unless>
+  <xacro:macro name="finger_collisions" params="prefix link_prefix lf" >
     <disable_collisions link1="${prefix}${link_prefix}${distal}" link2="${prefix}${link_prefix}${middle}" reason="Adjacent" />
     <disable_collisions link1="${prefix}${link_prefix}${distal}" link2="${prefix}${link_prefix}knuckle" reason="Never" />
@@ -147,11 +126,5 @@
     </xacro:if>
   </xacro:macro>
-  <xacro:macro name="thumb_collisions" params="prefix bio" >
-    <xacro:if value="${bio}">
-      <xacro:property name="distal" value="biotac"/>
-    </xacro:if>
-    <xacro:unless value="${bio}">
-      <xacro:property name="distal" value="distal"/>
-    </xacro:unless>
+  <xacro:macro name="thumb_collisions" params="prefix" >
     <disable_collisions link1="${prefix}forearm" link2="${prefix}thbase" reason="Never" />
     <disable_collisions link1="${prefix}forearm" link2="${prefix}th${distal}" reason="Never" />
@@ -184,21 +157,5 @@
   </xacro:macro>
   <!-- finger to other finger with a finger in between -->
-  <xacro:macro name="finger_farfinger_collisions" params="prefix link_prefix link_prefix2 lf bio bio2" >
-    <xacro:if value="${bio}">
-      <xacro:property name="distal" value="biotac"/>
-      <xacro:property name="middle" value="adapter"/>
-    </xacro:if>
-    <xacro:unless value="${bio}">
-      <xacro:property name="distal" value="distal"/>
-      <xacro:property name="middle" value="middle"/>
-    </xacro:unless>
-    <xacro:if value="${bio2}">
-      <xacro:property name="distal2" value="biotac"/>
-      <xacro:property name="middle2" value="adapter"/>
-      </xacro:if>
-    <xacro:unless value="${bio2}">
-      <xacro:property name="distal2" value="distal"/>
-      <xacro:property name="middle2" value="middle"/>
-    </xacro:unless>
+  <xacro:macro name="finger_farfinger_collisions" params="prefix link_prefix link_prefix2 lf" >
     <disable_collisions link1="${prefix}${link_prefix}${distal}" link2="${prefix}${link_prefix2}knuckle" reason="Never" />
     <disable_collisions link1="${prefix}${link_prefix}knuckle" link2="${prefix}${link_prefix2}${distal2}" reason="Never" />
@@ -225,21 +182,5 @@
   </xacro:macro>
   <!-- finger with two fingers in between (only ff-lf) -->
-  <xacro:macro name="first_little_collisions" params="prefix bio bio2" >
-    <xacro:if value="${bio}">
-      <xacro:property name="distal" value="biotac"/>
-      <xacro:property name="middle" value="adapter"/>
-    </xacro:if>
-    <xacro:unless value="${bio}">
-      <xacro:property name="distal" value="distal"/>
-      <xacro:property name="middle" value="middle"/>
-    </xacro:unless>
-    <xacro:if value="${bio2}">
-      <xacro:property name="distal2" value="biotac"/>
-      <xacro:property name="middle2" value="adapter"/>
-      </xacro:if>
-    <xacro:unless value="${bio2}">
-      <xacro:property name="distal2" value="distal"/>
-      <xacro:property name="middle2" value="middle"/>
-    </xacro:unless>
+  <xacro:macro name="first_little_collisions" params="prefix" >
     <disable_collisions link1="${prefix}ff${distal}" link2="${prefix}lfknuckle" reason="Never" />
     <disable_collisions link1="${prefix}ff${distal}" link2="${prefix}lfproximal" reason="Never" />
@@ -261,21 +202,5 @@
   </xacro:macro>
    <!-- finger next to other finger -->
-   <xacro:macro name="finger_closefinger_collisions" params="prefix link_prefix link_prefix2 lf bio bio2" >
-     <xacro:if value="${bio}">
-      <xacro:property name="distal" value="biotac"/>
-      <xacro:property name="middle" value="adapter"/>
-    </xacro:if>
-    <xacro:unless value="${bio}">
-      <xacro:property name="distal" value="distal"/>
-      <xacro:property name="middle" value="middle"/>
-    </xacro:unless>
-    <xacro:if value="${bio2}">
-      <xacro:property name="distal2" value="biotac"/>
-      <xacro:property name="middle2" value="adapter"/>
-      </xacro:if>
-    <xacro:unless value="${bio2}">
-      <xacro:property name="distal2" value="distal"/>
-      <xacro:property name="middle2" value="middle"/>
-    </xacro:unless>
+   <xacro:macro name="finger_closefinger_collisions" params="prefix link_prefix link_prefix2 lf" >
     <disable_collisions link1="${prefix}${link_prefix}${distal}" link2="${prefix}${link_prefix2}knuckle" reason="Never" />
     <disable_collisions link1="${prefix}${link_prefix}knuckle" link2="${prefix}${link_prefix2}${distal2}" reason="Never" />
@@ -294,19 +219,5 @@
   </xacro:macro>
    <!-- finger to thumb, far is 1 if at least one finger is in between -->
-   <xacro:macro name="finger_thumb_collisions" params="prefix link_prefix far lf thbio bio" >
-    <xacro:if value="${thbio}">
-      <xacro:property name="thdistal" value="thbiotac"/>
-    </xacro:if>
-    <xacro:unless value="${thbio}">
-      <xacro:property name="thdistal" value="thdistal"/>
-    </xacro:unless>
-    <xacro:if value="${bio}">
-      <xacro:property name="distal" value="biotac"/>
-      <xacro:property name="middle" value="adapter"/>
-      </xacro:if>
-    <xacro:unless value="${bio}">
-      <xacro:property name="distal" value="distal"/>
-      <xacro:property name="middle" value="middle"/>
-    </xacro:unless>
+   <xacro:macro name="finger_thumb_collisions" params="prefix link_prefix far lf" >
     <disable_collisions link1="${prefix}${link_prefix}${distal}" link2="${prefix}thbase" reason="Never" />
     <disable_collisions link1="${prefix}${link_prefix}${distal}" link2="${prefix}thhub" reason="Never" />

File: sr_moveit_hand_config/config/shadowhands.srdf.xacro (robot description, xacro)
@@ -2,4 +2,5 @@
 <robot xmlns:xacro="http://www.ros.org/wiki/xacro" name="$(arg robot_name)">
   <xacro:include filename="$(find sr_moveit_hand_config)/config/shadowhand.srdf.xacro"/>
+  <xacro:arg name="prefix" default="rh_"/>
   <xacro:arg name="ff" default="1"/>
   <xacro:arg name="mf" default="1"/>
@@ -17,22 +18,60 @@
   <group name="shadow_hand">
     <xacro:if value="$(arg th)">
-      <xacro:thumblinks prefix="" bio="$(arg th_bio)"/>
+      <xacro:if value="$(arg th_bio)">
+        <xacro:property name="distal" value="biotac"/>
+      </xacro:if>
+      <xacro:unless value="$(arg th_bio)">
+        <xacro:property name="distal" value="distal"/>
+      </xacro:unless>
+      <xacro:thumblinks prefix="" />
       <xacro:thumbjoints prefix=""/>
     </xacro:if>
     <xacro:if value="$(arg ff)">
-      <xacro:fingerlinks prefix="" link_prefix="ff" bio="$(arg ff_bio)" lf="0"/>
+      <xacro:if value="$(arg ff_bio)">
+        <xacro:property name="distal" value="biotac"/>
+        <xacro:property name="middle" value="adapter"/>
+      </xacro:if>
+      <xacro:unless value="$(arg ff_bio)">
+        <xacro:property name="distal" value="distal"/>
+        <xacro:property name="middle" value="middle"/>
+      </xacro:unless>
+      <xacro:fingerlinks prefix="" link_prefix="ff" lf="0"/>
       <xacro:fingerjoints prefix="" joint_prefix="FF" lf="0"/>
     </xacro:if>
     <xacro:if value="$(arg mf)">
-      <xacro:fingerlinks prefix="" link_prefix="mf" bio="$(arg mf_bio)" lf="0"/>
+      <xacro:if value="$(arg mf_bio)">
+        <xacro:property name="distal" value="biotac"/>
+        <xacro:property name="middle" value="adapter"/>
+      </xacro:if>
+      <xacro:unless value="$(arg mf_bio)">
+        <xacro:property name="distal" value="distal"/>
+        <xacro:property name="middle" value="middle"/>
+      </xacro:unless>
+      <xacro:fingerlinks prefix="" link_prefix="mf" lf="0"/>
       <xacro:fingerjoints prefix="" joint_prefix="MF" lf="0"/>
     </xacro:if>
     <xacro:if value="$(arg rf)">
-      <xacro:fingerlinks prefix="" link_prefix="rf" bio="$(arg rf_bio)" lf="0"/>
+      <xacro:if value="$(arg rf_bio)">
+        <xacro:property name="distal" value="biotac"/>
+        <xacro:property name="middle" value="adapter"/>
+      </xacro:if>
+      <xacro:unless value="$(arg rf_bio)">
+        <xacro:property name="distal" value="distal"/>
+        <xacro:property name="middle" value="middle"/>
+      </xacro:unless>
+      <xacro:fingerlinks prefix="" link_prefix="rf" lf="0"/>
       <xacro:fingerjoints prefix="" joint_prefix="RF" lf="0"/>
     </xacro:if>
     <xacro:unless value="$(arg is_lite)">
       <xacro:if value="$(arg lf)">
-        <xacro:fingerlinks prefix="" link_prefix="lf" bio="$(arg lf_bio)" lf="1"/>
+        <xacro:if value="$(arg lf_bio)">
+          <xacro:property name="distal" value="biotac"/>
+          <xacro:property name="middle" value="adapter"/>
+        </xacro:if>
+        <xacro:unless value="$(arg lf_bio)">
+          <xacro:property name="distal" value="distal"/>
+          <xacro:property name="middle" value="middle"/>
+        </xacro:unless>
+        <xacro:fingerlinks prefix="" link_prefix="lf" lf="1"/>
         <xacro:fingerjoints prefix="" joint_prefix="LF" lf="1"/>
       </xacro:if>
@@ -266,34 +305,110 @@
   <!-- single fingers collision -->
   <xacro:if value="$(arg ff)">
-     <xacro:finger_collisions prefix="" link_prefix="ff" lf="0" bio="$(arg ff_bio)"/>
+    <xacro:if value="$(arg ff_bio)">
+      <xacro:property name="distal" value="biotac"/>
+      <xacro:property name="middle" value="adapter"/>
+    </xacro:if>
+    <xacro:unless value="$(arg ff_bio)">
+      <xacro:property name="distal" value="distal"/>
+      <xacro:property name="middle" value="middle"/>
+    </xacro:unless>
+    <xacro:finger_collisions prefix="" link_prefix="ff" lf="0" />
   </xacro:if>
   <xacro:if value="$(arg mf)">
-     <xacro:finger_collisions prefix="" link_prefix="mf" lf="0" bio="$(arg mf_bio)"/>
+    <xacro:if value="$(arg mf_bio)">
+      <xacro:property name="distal" value="biotac"/>
+      <xacro:property name="middle" value="adapter"/>
+    </xacro:if>
+    <xacro:unless value="$(arg mf_bio)">
+      <xacro:property name="distal" value="distal"/>
+      <xacro:property name="middle" value="middle"/>
+    </xacro:unless>
+    <xacro:finger_collisions prefix="" link_prefix="mf" lf="0" />
   </xacro:if>
   <xacro:if value="$(arg rf)">
-     <xacro:finger_collisions prefix="" link_prefix="rf" lf="0" bio="$(arg rf_bio)"/>
+    <xacro:if value="$(arg rf_bio)">
+      <xacro:property name="distal" value="biotac"/>
+      <xacro:property name="middle" value="adapter"/>
+    </xacro:if>
+    <xacro:unless value="$(arg rf_bio)">
+      <xacro:property name="distal" value="distal"/>
+      <xacro:property name="middle" value="middle"/>
+    </xacro:unless>
+    <xacro:finger_collisions prefix="" link_prefix="rf" lf="0" />
   </xacro:if>
   <xacro:unless value="$(arg is_lite)">
     <xacro:if value="$(arg lf)">
-       <xacro:finger_collisions prefix="" link_prefix="lf" lf="1" bio="$(arg lf_bio)"/>
+      <xacro:if value="$(arg lf_bio)">
+        <xacro:property name="distal" value="biotac"/>
+        <xacro:property name="middle" value="adapter"/>
+      </xacro:if>
+      <xacro:unless value="$(arg lf_bio)">
+        <xacro:property name="distal" value="distal"/>
+        <xacro:property name="middle" value="middle"/>
+      </xacro:unless>
+       <xacro:finger_collisions prefix="" link_prefix="lf" lf="1" />
     </xacro:if>
   </xacro:unless>
   <xacro:if value="$(arg th)">
-    <xacro:thumb_collisions prefix="" bio="$(arg th_bio)"/>
+    <xacro:if value="$(arg th_bio)">
+      <xacro:property name="distal" value="biotac"/>
+    </xacro:if>
+    <xacro:unless value="$(arg th_bio)">
+      <xacro:property name="distal" value="distal"/>
+    </xacro:unless>
+    <xacro:thumb_collisions prefix="" />
   </xacro:if>
   <!-- pairs with thumb for collision-->
   <xacro:if value="$(arg th)">
-    <xacro:if value="$(arg ff)">
-      <xacro:finger_thumb_collisions  prefix="" link_prefix="ff" far="0" lf="0" thbio="$(arg th_bio)" bio="$(arg ff_bio)"/>
-    </xacro:if>
-    <xacro:if value="$(arg mf)">
-      <xacro:finger_thumb_collisions  prefix="" link_prefix="mf" far="1" lf="0" thbio="$(arg th_bio)" bio="$(arg mf_bio)"/>
-    </xacro:if>
-    <xacro:if value="$(arg rf)">
-      <xacro:finger_thumb_collisions  prefix="" link_prefix="rf" far="1" lf="0" thbio="$(arg th_bio)" bio="$(arg rf_bio)"/>
-    </xacro:if>
-    <xacro:unless value="$(arg is_lite)">
-      <xacro:if value="$(arg lf)">
-          <xacro:finger_thumb_collisions  prefix="" link_prefix="lf" far="1" lf="1" thbio="$(arg th_bio)" bio="$(arg lf_bio)"/>
+    <xacro:if value="$(arg th_bio)">
+      <xacro:property name="thdistal" value="thbiotac"/>
+    </xacro:if>
+    <xacro:unless value="$(arg th_bio)">
+      <xacro:property name="thdistal" value="thdistal"/>
+    </xacro:unless>
+    <xacro:if value="$(arg ff)">
+      <xacro:if value="$(arg ff_bio)">
+        <xacro:property name="distal" value="biotac"/>
+        <xacro:property name="middle" value="adapter"/>
+      </xacro:if>
+      <xacro:unless value="$(arg ff_bio)">
+        <xacro:property name="distal" value="distal"/>
+        <xacro:property name="middle" value="middle"/>
+      </xacro:unless>
+      <xacro:finger_thumb_collisions  prefix="" link_prefix="ff" far="0" lf="0" />
+    </xacro:if>
+    <xacro:if value="$(arg mf)">
+      <xacro:if value="$(arg mf_bio)">
+        <xacro:property name="distal" value="biotac"/>
+        <xacro:property name="middle" value="adapter"/>
+      </xacro:if>
+      <xacro:unless value="$(arg mf_bio)">
+        <xacro:property name="distal" value="distal"/>
+        <xacro:property name="middle" value="middle"/>
+      </xacro:unless>
+      <xacro:finger_thumb_collisions  prefix="" link_prefix="mf" far="1" lf="0" />
+    </xacro:if>
+    <xacro:if value="$(arg rf)">
+      <xacro:if value="$(arg rf_bio)">
+        <xacro:property name="distal" value="biotac"/>
+        <xacro:property name="middle" value="adapter"/>
+      </xacro:if>
+      <xacro:unless value="$(arg rf_bio)">
+        <xacro:property name="distal" value="distal"/>
+        <xacro:property name="middle" value="middle"/>
+      </xacro:unless>
+      <xacro:finger_thumb_collisions  prefix="" link_prefix="rf" far="1" lf="0" />
+    </xacro:if>
+    <xacro:unless value="$(arg is_lite)">
+      <xacro:if value="$(arg lf)">
+          <xacro:if value="$(arg lf_bio)">
+            <xacro:property name="distal" value="biotac"/>
+            <xacro:property name="middle" value="adapter"/>
+          </xacro:if>
+          <xacro:unless value="$(arg lf_bio)">
+            <xacro:property name="distal" value="distal"/>
+            <xacro:property name="middle" value="middle"/>
+          </xacro:unless>
+          <xacro:finger_thumb_collisions  prefix="" link_prefix="lf" far="1" lf="1" />
       </xacro:if>
     </xacro:unless>
@@ -302,12 +417,60 @@
   <xacro:if value="$(arg ff)">
     <xacro:if value="$(arg mf)">
-      <xacro:finger_closefinger_collisions prefix="" link_prefix="ff" link_prefix2="mf"  lf="0" bio="$(arg ff_bio)" bio2="$(arg mf_bio)"/>
-    </xacro:if>
-    <xacro:if value="$(arg rf)">
-      <xacro:finger_farfinger_collisions prefix="" link_prefix="ff" link_prefix2="rf"  lf="0" bio="$(arg ff_bio)" bio2="$(arg rf_bio)"/>
-    </xacro:if>
-    <xacro:unless value="$(arg is_lite)">
-      <xacro:if value="$(arg lf)">
-        <xacro:first_little_collisions prefix="" bio="$(arg ff_bio)" bio2="$(arg lf_bio)" />
+      <xacro:if value="$(arg ff_bio)">
+        <xacro:property name="distal" value="biotac"/>
+        <xacro:property name="middle" value="adapter"/>
+      </xacro:if>
+      <xacro:unless value="$(arg ff_bio)">
+        <xacro:property name="distal" value="distal"/>
+        <xacro:property name="middle" value="middle"/>
+      </xacro:unless>
+      <xacro:if value="$(arg mf_bio)">
+        <xacro:property name="distal2" value="biotac"/>
+        <xacro:property name="middle2" value="adapter"/>
+        </xacro:if>
+      <xacro:unless value="$(arg mf_bio)">
+        <xacro:property name="distal2" value="distal"/>
+        <xacro:property name="middle2" value="middle"/>
+      </xacro:unless>
+      <xacro:finger_closefinger_collisions prefix="" link_prefix="ff" link_prefix2="mf"  lf="0"/>
+    </xacro:if>
+    <xacro:if value="$(arg rf)">
+      <xacro:if value="$(arg ff_bio)">
+        <xacro:property name="distal" value="biotac"/>
+        <xacro:property name="middle" value="adapter"/>
+      </xacro:if>
+      <xacro:unless value="$(arg ff_bio)">
+        <xacro:property name="distal" value="distal"/>
+        <xacro:property name="middle" value="middle"/>
+      </xacro:unless>
+      <xacro:if value="$(arg rf_bio)">
+        <xacro:property name="distal2" value="biotac"/>
+        <xacro:property name="middle2" value="adapter"/>
+        </xacro:if>
+      <xacro:unless value="$(arg rf_bio)">
+        <xacro:property name="distal2" value="distal"/>
+        <xacro:property name="middle2" value="middle"/>
+      </xacro:unless>
+      <xacro:finger_farfinger_collisions prefix="" link_prefix="ff" link_prefix2="rf"  lf="0" />
+    </xacro:if>
+    <xacro:unless value="$(arg is_lite)">
+      <xacro:if value="$(arg lf)">
+        <xacro:if value="$(arg ff_bio)">
+          <xacro:property name="distal" value="biotac"/>
+          <xacro:property name="middle" value="adapter"/>
+        </xacro:if>
+        <xacro:unless value="$(arg ff_bio)">
+          <xacro:property name="distal" value="distal"/>
+          <xacro:property name="middle" value="middle"/>
+        </xacro:unless>
+        <xacro:if value="$(arg lf_bio)">
+          <xacro:property name="distal2" value="biotac"/>
+          <xacro:property name="middle2" value="adapter"/>
+          </xacro:if>
+        <xacro:unless value="$(arg lf_bio)">
+          <xacro:property name="distal2" value="distal"/>
+          <xacro:property name="middle2" value="middle"/>
+        </xacro:unless>
+        <xacro:first_little_collisions prefix="" />
       </xacro:if>
     </xacro:unless>
@@ -315,9 +478,41 @@
   <xacro:if value="$(arg mf)">
     <xacro:if value="$(arg rf)">
-      <xacro:finger_closefinger_collisions prefix="" link_prefix="mf" link_prefix2="rf"  lf="0" bio="$(arg mf_bio)" bio2="$(arg rf_bio)"/>
-    </xacro:if>
-    <xacro:unless value="$(arg is_lite)">
-      <xacro:if value="$(arg lf)">
-        <xacro:finger_farfinger_collisions prefix="" link_prefix="mf" link_prefix2="lf"  lf="1" bio="$(arg mf_bio)" bio2="$(arg lf_bio)"/>
+      <xacro:if value="$(arg mf_bio)">
+        <xacro:property name="distal" value="biotac"/>
+        <xacro:property name="middle" value="adapter"/>
+      </xacro:if>
+      <xacro:unless value="$(arg mf_bio)">
+        <xacro:property name="distal" value="distal"/>
+        <xacro:property name="middle" value="middle"/>
+      </xacro:unless>
+      <xacro:if value="$(arg rf_bio)">
+        <xacro:property name="distal2" value="biotac"/>
+        <xacro:property name="middle2" value="adapter"/>
+        </xacro:if>
+      <xacro:unless value="$(arg rf_bio)">
+        <xacro:property name="distal2" value="distal"/>
+        <xacro:property name="middle2" value="middle"/>
+      </xacro:unless>
+      <xacro:finger_closefinger_collisions prefix="" link_prefix="mf" link_prefix2="rf"  lf="0" />
+    </xacro:if>
+    <xacro:unless value="$(arg is_lite)">
+      <xacro:if value="$(arg lf)">
+        <xacro:if value="$(arg mf_bio)">
+          <xacro:property name="distal" value="biotac"/>
+          <xacro:property name="middle" value="adapter"/>
+        </xacro:if>
+        <xacro:unless value="$(arg mf_bio)">
+          <xacro:property name="distal" value="distal"/>
+          <xacro:property name="middle" value="middle"/>
+        </xacro:unless>
+        <xacro:if value="$(arg lf_bio)">
+          <xacro:property name="distal2" value="biotac"/>
+          <xacro:property name="middle2" value="adapter"/>
+          </xacro:if>
+        <xacro:unless value="$(arg lf_bio)">
+          <xacro:property name="distal2" value="distal"/>
+          <xacro:property name="middle2" value="middle"/>
+        </xacro:unless>
+        <xacro:finger_farfinger_collisions prefix="" link_prefix="mf" link_prefix2="lf"  lf="1" />
       </xacro:if>
     </xacro:unless>
@@ -326,5 +521,21 @@
     <xacro:unless value="$(arg is_lite)">
       <xacro:if value="$(arg lf)">
-        <xacro:finger_closefinger_collisions prefix="" link_prefix="rf" link_prefix2="lf"  lf="1" bio="$(arg rf_bio)" bio2="$(arg lf_bio)"/>
+        <xacro:if value="$(arg rf_bio)">
+          <xacro:property name="distal" value="biotac"/>
+          <xacro:property name="middle" value="adapter"/>
+        </xacro:if>
+        <xacro:unless value="$(arg rf_bio)">
+          <xacro:property name="distal" value="distal"/>
+          <xacro:property name="middle" value="middle"/>
+        </xacro:unless>
+        <xacro:if value="$(arg lf_bio)">
+          <xacro:property name="distal2" value="biotac"/>
+          <xacro:property name="middle2" value="adapter"/>
+          </xacro:if>
+        <xacro:unless value="$(arg lf_bio)">
+          <xacro:property name="distal2" value="distal"/>
+          <xacro:property name="middle2" value="middle"/>
+        </xacro:unless>
+        <xacro:finger_closefinger_collisions prefix="" link_prefix="rf" link_prefix2="lf"  lf="1" />
       </xacro:if>
     </xacro:unless>
